File: PCBs/draadlossdeurbel.kicad_sch (KiCad schematic)
At the start: 8 parts

Commit message: bijgewerkt
Parts:
- added U?: SN76489, w_pth_circuits:dil_16-300_socket, symbol easylab4kids:SN76489
Connections:
- net GND: now also U?.8 (GND)
- net VCC: now also U?.16 (VCC)
- net CLOCK: now reaches U?.2 (A0)
- net CLOCK: now also U?.3 (QD)
- net D2: now reaches U?.1 (QB)
Changed lines of the file:
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@@
+    (stroke (width 0) (type default) (color 0 0 0 0))
+  )
+  (wire (pts (xy 177.8 54.61) (xy 184.15 54.61))
     (stroke (width 0) (type default) (color 0 0 0 0))
   )
@@
     (stroke (width 0) (type default) (color 0 0 0 0))
   )
+  (wire (pts (xy 210.82 59.69) (xy 218.44 59.69))
+    (stroke (width 0) (type default) (color 0 0 0 0))
+  )
   (wire (pts (xy 62.23 24.13) (xy 140.97 24.13))
     (stroke (width 0) (type default) (color 0 0 0 0))
@@
     (stroke (width 0) (type default) (color 0 0 0 0))
   )
+  (wire (pts (xy 177.8 49.53) (xy 184.15 49.53))
+    (stroke (width 0) (type default) (color 0 0 0 0))
+  )
+  (wire (pts (xy 151.13 45.72) (xy 160.02 45.72))
+    (stroke (width 0) (type default) (color 0 0 0 0))
+  )
   (wire (pts (xy 107.95 88.9) (xy 109.22 88.9))
     (stroke (width 0) (type default) (color 0 0 0 0))
   )
+  (wire (pts (xy 74.93 41.91) (xy 82.55 41.91))
+    (stroke (width 0) (type default) (color 0 0 0 0))
+  )
+  (wire (pts (xy 210.82 62.23) (xy 218.44 62.23))
+    (stroke (width 0) (type default) (color 0 0 0 0))
+  )
+  (wire (pts (xy 177.8 64.77) (xy 184.15 64.77))
+    (stroke (width 0) (type default) (color 0 0 0 0))
+  )
+  (wire (pts (xy 210.82 52.07) (xy 218.44 52.07))
+    (stroke (width 0) (type default) (color 0 0 0 0))
+  )
   (wire (pts (xy 96.52 88.9) (xy 100.33 88.9))
     (stroke (width 0) (type default) (color 0 0 0 0))
@@
     (stroke (width 0) (type default) (color 0 0 0 0))
   )
+  (wire (pts (xy 210.82 49.53) (xy 218.44 49.53))
+    (stroke (width 0) (type default) (color 0 0 0 0))
+  )
   (wire (pts (xy 116.84 93.98) (xy 116.84 97.79))
     (stroke (width 0) (type default) (color 0 0 0 0))
   )
+  (wire (pts (xy 177.8 57.15) (xy 184.15 57.15))
+    (stroke (width 0) (type default) (color 0 0 0 0))
+  )
+  (wire (pts (xy 177.8 52.07) (xy 184.15 52.07))
+    (stroke (width 0) (type default) (color 0 0 0 0))
+  )
+  (wire (pts (xy 177.8 59.69) (xy 184.15 59.69))
+    (stroke (width 0) (type default) (color 0 0 0 0))
+  )
+  (wire (pts (xy 177.8 62.23) (xy 184.15 62.23))
+    (stroke (width 0) (type default) (color 0 0 0 0))
+  )
   (wire (pts (xy 86.36 77.47) (xy 86.36 81.28))
     (stroke (width 0) (type default) (color 0 0 0 0))
   )
+  (wire (pts (xy 177.8 46.99) (xy 184.15 46.99))
+    (stroke (width 0) (type default) (color 0 0 0 0))
+  )
+  (wire (pts (xy 210.82 57.15) (xy 218.44 57.15))
+    (stroke (width 0) (type default) (color 0 0 0 0))
+  )
   (wire (pts (xy 111.76 101.6) (xy 86.36 101.6))
     (stroke (width 0) (type default) (color 0 0 0 0))
   )
+  (wire (pts (xy 210.82 54.61) (xy 218.44 54.61))
+    (stroke (width 0) (type default) (color 0 0 0 0))
+  )
   (wire (pts (xy 86.36 96.52) (xy 86.36 101.6))
     (stroke (width 0) (type default) (color 0 0 0 0))
   )
+  (wire (pts (xy 151.13 50.8) (xy 160.02 50.8))
+    (stroke (width 0) (type default) (color 0 0 0 0))
+  )
+  (wire (pts (xy 210.82 46.99) (xy 218.44 46.99))
+    (stroke (width 0) (type default) (color 0 0 0 0))
+  )
   (label "LED" (at 116.84 96.52 90)
     (effects (font (size 0.66 0.66)) (justify left bottom))
   )
+  (label "D2" (at 153.67 45.72 0)
+    (effects (font (size 0.66 0.66)) (justify left bottom))
+  )
   (label "VCC" (at 140.97 36.83 90)
     (effects (font (size 0.66 0.66)) (justify left bottom))
@@
     (effects (font (size 0.66 0.66)) (justify left bottom))
   )
+  (label "CLOCK" (at 153.67 50.8 0)
+    (effects (font (size 0.66 0.66)) (justify left bottom))
+  )
   (label "GND" (at 111.76 116.84 90)
+    (effects (font (size 0.66 0.66)) (justify left bottom))
+  )
+  (label "VCC" (at 212.09 46.99 0)
+    (effects (font (size 0.66 0.66)) (justify left bottom))
+  )
+  (label "CLOCK" (at 76.2 41.91 0)
     (effects (font (size 0.66 0.66)) (justify left bottom))
   )
   (label "AUDIO_UIT" (at 96.52 88.9 0)
     (effects (font (size 0.5 0.5)) (justify left bottom))
+  )
+  (label "GND" (at 182.88 64.77 180)
+    (effects (font (size 0.66 0.66)) (justify right bottom))
   )
   (symbol (lib_id "power:VCC") (at 86.36 77.47 0) (unit 1)
@@
     (pin "9")
   )
-  (symbol (lib_id "power:GND") (at 64.77 81.28 0) (unit 1)
-    (in_bom yes) (on_board yes)
-    (property "Reference" "#PWR0103" (id 0) (at 64.77 87.63 0)
-      (effects (font (size 0.66 0.66)) hide)
-    )
-    (property "Value" "GND" (id 1) (at 66.04 85.09 0)
-      (effects (font (size 0.66 0.66)) (justify right))
-    )
-    (property "Footprint" "" (id 2) (at 64.77 81.28 0)
-      (effects (font (size 0.66 0.66)) hide)
-    )
-    (property "Datasheet" "" (id 3) (at 64.77 81.28 0)
-      (effects (font (size 0.66 0.66)) hide)
-    )
-    (pin "1")
-  )
-  (symbol (lib_id "74xx:74HC595") (at 140.97 53.34 0) (unit 1)
-    (in_bom yes) (on_board yes) (fields_autoplaced)
-    (property "Reference" "U?" (id 0) (at 142.9894 36.83 0)
-      (effects (font (size 1.27 1.27)) (justify left))
-    )
-    (property "Value" "74HC595" (id 1) (at 142.9894 39.37 0)
-      (effects (font (size 0.66 0.66)) (justify left))
-    )
-    (property "Footprint" "" (id 2) (at 140.97 53.34 0)
-      (effects (font (size 1.27 1.27)) hide)
-    )
-    (property "Datasheet" "http://www.ti.com/lit/ds/symlink/sn74hc595.pdf" (id 3) (at 140.97 53.34 0)
-      (effects (font (size 1.27 1.27)) hide)
+  (symbol (lib_id "easylab4kids:SN76489") (at 198.12 55.88 0) (unit 1)
+    (in_bom yes) (on_board yes)
+    (property "Reference" "U?" (id 0) (at 198.12 41.91 0)
+      (effects (font (size 1.524 1.524)))
+    )
+    (property "Value" "SN76489" (id 1) (at 198.12 68.58 0)
+      (effects (font (size 1.524 1.524)))
+    )
+    (property "Footprint" "w_pth_circuits:dil_16-300_socket" (id 2) (at 198.12 63.5 0)
+      (effects (font (size 1.524 1.524)) hide)
+    )
+    (property "Datasheet" "" (id 3) (at 198.12 63.5 0)
+      (effects (font (size 1.524 1.524)) hide)
     )
     (pin "1")
@@
     (pin "9")
   )
+  (symbol (lib_id "power:GND") (at 64.77 81.28 0) (unit 1)
+    (in_bom yes) (on_board yes)
+    (property "Reference" "#PWR0103" (id 0) (at 64.77 87.63 0)
+      (effects (font (size 0.66 0.66)) hide)
+    )
+    (property "Value" "GND" (id 1) (at 66.04 85.09 0)
+      (effects (font (size 0.66 0.66)) (justify right))
+    )
+    (property "Footprint" "" (id 2) (at 64.77 81.28 0)
+      (effects (font (size 0.66 0.66)) hide)
+    )
+    (property "Datasheet" "" (id 3) (at 64.77 81.28 0)
+      (effects (font (size 0.66 0.66)) hide)
+    )
+    (pin "1")
+  )
+  (symbol (lib_id "74xx:74HC595") (at 140.97 53.34 0) (unit 1)
+    (in_bom yes) (on_board yes) (fields_autoplaced)
+    (property "Reference" "U?" (id 0) (at 142.9894 36.83 0)
+      (effects (font (size 1.27 1.27)) (justify left))
+    )
+    (property "Value" "74HC595" (id 1) (at 142.9894 39.37 0)
+      (effects (font (size 0.66 0.66)) (justify left))
+    )
+    (property "Footprint" "" (id 2) (at 140.97 53.34 0)
+      (effects (font (size 1.27 1.27)) hide)
+    )
+    (property "Datasheet" "http://www.ti.com/lit/ds/symlink/sn74hc595.pdf" (id 3) (at 140.97 53.34 0)
+      (effects (font (size 1.27 1.27)) hide)
+    )
+    (pin "1")
+    (pin "10")
+    (pin "11")
+    (pin "12")
+    (pin "13")
+    (pin "14")
+    (pin "15")
+    (pin "16")
+    (pin "2")
+    (pin "3")
+    (pin "4")
+    (pin "5")
+    (pin "6")
+    (pin "7")
+    (pin "8")
+    (pin "9")
+  )
   (sheet_instances
     (path "/" (page "1"))
@@
       (reference "U?") (unit 1) (value "WeMos_D1_mini") (footprint "Module:WEMOS_D1_mini_light")
     )
+    (path "/d5b94a30-6408-43d1-8792-f8b177f4e785"
+      (reference "U?") (unit 1) (value "SN76489") (footprint "w_pth_circuits:dil_16-300_socket")
+    )
     (path "/fc4733a3-c200-4f8e-9f63-f3b7c6201473"

Commit message: bijgewerkt
Parts:
- BZ1: renamed from BZ?; value Buzzer -> Zoemer
- gave numbers to parts that had none: 7
- renumbered R to R2
Connections:
- net GND: now also U2.2 (-), U3.13 (~{OE})
- net AUDIO: now reaches U2.3 (+)
- net AUDIO: now also U4.7 (AUDIO_OUT)
- net DeepSleep: now reaches U1.1 (~{RST})
- net DeepSleep: now also U1.3 (D0)
- net Qc: now reaches U4.1 (D2)
- net Qc: now also U3.2 (QC)
- net Qh: now reaches U4.10 (D7)
- net Qh: now also U3.7 (QH)
- net Qg: now reaches U4.11 (D6)
- net Qg: now also U3.6 (QG)
- net Qf: now reaches U4.12 (D5)
- net Qf: now also U3.5 (QF)
- net Qe: now reaches U4.13 (D4)
- net Qe: now also U3.4 (QE)
- net PWM_CLK: now reaches U4.14 (CLOCK)
- net PWM_CLK: now also U1.2 (A0)
- net Qd: now reaches U4.15 (D3)
- net Qd: now also U3.3 (QD)
- net Qb: now reaches U4.2 (D1)
- net Qa: now reaches U4.3 (D0)
- net Qa: now also U3.15 (QA)
- net RCLCK: now reaches U3.11 (SRCLK)
- removed net CLOCK: U1.2 (A0), U3.3 (QD)
- no-connect marks 0 -> 4

Commit message: bijgewerkt
Parts:
- removed Q1: BC337, Package_TO_SOT_THT:TO-92_Inline, symbol Transistor_BJT:BC337
- added C1: 10uF, symbol Device:C_Polarized_Small
- added C2: 250uF, symbol Device:C_Polarized_US
- added C3: C, symbol Device:C
- added J1: AudioJack4_Ground, symbol Connector:AudioJack4_Ground
- added Q1: BC161, Package_TO_SOT_THT:TO-39-3, symbol Transistor_BJT:BC161
Connections:
- net RCLCK is gone; now on net SRCLK: U3.11 (SRCLK)
- net AUDIO_UIT: now also C2.1; no longer R1.1
- net GND: now also D1.1 (K), U2.7 (BYPASS), C3.1, C3.2, J1.G
- net LED: now also U1.12 (D3)
- net VCC: now also U3.10 (~{SRCLR})
- net Zoemer: now reaches BZ1.1 (-)
- net Zoemer: now also Q1.3 (C); no longer D1.1 (K)
- net at U2.1 (GAIN): now also C1.1
- net at U2.8 (GAIN): now also C1.2
- net at R1.2: now also Q1.1 (E)
- net GeluidAanUit: now reaches U1.11 (D4)
- net GeluidAanUit: now also Q1.2 (B)
- net SRCLK: now reaches U1.4 (SCK/D5)
- net MISO: now reaches U1.5 (MISO/D6)
- net MOSI: now reaches U1.6 (MOSI/D7)
- net MOSI: now also U3.14 (SER)
- net CS: now reaches U1.7 (CS/D8)
- net RCLK: now reaches U3.12 (RCLK)
- net AUDIO renamed SN76489_geluid
- new net: C2.2, R1.1
Other:
- note added: "Wireless Doorbell 0.0.1 Work-in-progress!!"
- moved on the sheet: BZ1, D1, R1, R2, U2

Commit message: bijgewerkt
Parts:
- removed C1: 10uF, symbol Device:C_Polarized_Small
- added C4, C?: 0.05uF, symbol Device:C
- added R3: R1k, symbol Device:R
- C3: value C -> 10uF
Connections:
- net AUDIO_UIT: now also C4.2
- net GND: now also U4.6 (~{OE}), C4.1
- net at U2.1 (GAIN): now also R3.1
- net at U2.8 (GAIN): now also C?.1
- net WE: now reaches U1.14 (SCL/D1)
- net WE: now also U4.5 (~{WE})
- new net: C?.2, R3.2
Other:
- moved on the sheet: BZ1

Commit message: bijgewerkt
Parts:
- D1: value LED -> LED-R
Changed lines of the file:
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@@
   (symbol (lib_id "Device:LED") (at 93.98 55.88 90) (unit 1)
     (in_bom yes) (on_board yes) (fields_autoplaced)
-    (property "Reference" "D1" (id 0) (at 97.79 56.1974 90)
-      (effects (font (size 0.66 0.66)) (justify right))
-    )
-    (property "Value" "LED" (id 1) (at 97.79 58.7374 90)
+    (property "Reference" "D1" (id 0) (at 97.79 56.8325 90)
+      (effects (font (size 0.66 0.66)) (justify right))
+    )
+    (property "Value" "LED-R" (id 1) (at 97.79 59.3725 90)
       (effects (font (size 0.66 0.66)) (justify right))
     )
@@
     )
     (path "/37e60867-fcfc-4a83-95aa-23a504162dab"
-      (reference "D1") (unit 1) (value "LED") (footprint "")
+      (reference "D1") (unit 1) (value "LED-R") (footprint "")
     )
     (path "/2d610dfd-d102-495c-b231-c5a0cd02efc6"

Commit message: bijgewerkt
Parts:
- added C5: C, symbol Device:C
- added J?: VCC, symbol Connector_Generic:Conn_01x01
- added J?: Conn_01x02, symbol Connector_Generic:Conn_01x02
- added R? (x4): R100, symbol Device:R
- added U5: TP4056, symbol EasyLab4Kids:TP4056
- gave numbers to parts that had none: 1
Connections:
- net GND: now also C5.2, J?.2 (Pin_2), R?.1, R?.2, R?.2, R?.2, U5.3 (GND)
- new net: R?.1, U5.2 (PROG)
- new net: R?.1, R?.2, U5.4 (VCC)
- new net: J?.1 (Pin_1), R?.1
- new net BAT+: C5.1, J?.1 (Pin_1), U5.5 (BAT)
Other:
- note added: "Batterij power management"
- note added: "Geluid output"
- moved on the sheet: BZ1, C1, C2, C3, C4, J1, Q1, R1, R3, U2

Commit message: bijgewerkt
Parts:
- removed C5: C, symbol Device:C
- removed J1: AudioJack4_Ground, symbol Connector:AudioJack4_Ground
- removed J?: VCC, symbol Connector_Generic:Conn_01x01
- removed J?: Conn_01x02, symbol Connector_Generic:Conn_01x02
- removed R? (x4): R100, symbol Device:R
- removed U5: TP4056, symbol EasyLab4Kids:TP4056
- added BT1: Battery_Cell, symbol Device:Battery_Cell
- added U5: TP4056-breakout, symbol EasyLab4Kids:TP4056-breakout
Connections:
- net GND: now also U5. (OUT-)
- net VCC: now also U5. (OUT-)
- new net: BT1.1 (+), U5. (OUT-)
- new net: BT1.2 (-), U5. (OUT-)
Other:
- note added: "Zonnenpaneel oplader"
- note removed: "Batterij power management"

Commit message: bijgewerkt
Connections:
- net LED: now also U3.9 (QH'); no longer U1.12 (D3)
- net SRCLK: no longer U1.4 (SCK/D5)
- net CS renamed Latch
- net MISO renamed SCK
- no-connect marks 4 -> 3
Other:
- moved on the sheet: D1, R2, U4
